Commit message: fixed units

File: src/navvis_description/urdf/robot.xacro (robot description, xacro)
@@ -27,5 +27,5 @@
             <origin xyz="0.0 0.0 0.0" rpy="0.0 0.0 0.0" />
             <geometry>
-                <box size="0.62 0.62 0.87" />
+                <box size="0.062 0.062 0.087" />
             </geometry>
         </visual>
@@ -33,5 +33,5 @@
             <origin xyz="0.0 0.0 0.0" rpy="0.0 0.0 0.0" />
             <geometry>
-                <box size="0.62 0.62 0.87" />
+                <box size="0.062 0.062 0.087" />
             </geometry>
         </collision>
@@ -46,5 +46,5 @@
             <origin xyz="0.0 0.0 0.0" rpy="0.0 0.0 0.0" />
             <geometry>
-                <box size="0.62 0.62 0.87" />
+                <box size="0.062 0.062 0.087" />
             </geometry>
         </visual>
@@ -52,5 +52,5 @@
             <origin xyz="0.0 0.0 0.0" rpy="0.0 0.0 0.0" />
             <geometry>
-                <box size="0.62 0.62 0.87" />
+                <box size="0.062 0.062 0.087" />
             </geometry>
         </collision>
@@ -65,5 +65,5 @@
             <origin xyz="0.0 0.0 0.0" rpy="0.0 0.0 0.0" />
             <geometry>
-                <box size="0.62 0.62 0.87" />
+                <box size="0.062 0.062 0.087" />
             </geometry>
         </visual>
@@ -71,5 +71,5 @@
             <origin xyz="0.0 0.0 0.0" rpy="0.0 0.0 0.0" />
             <geometry>
-                <box size="0.62 0.62 0.87" />
+                <box size="0.062 0.062 0.087" />
             </geometry>
         </collision>
@@ -84,5 +84,5 @@
             <origin xyz="0.0 0.0 0.0" rpy="0.0 0.0 0.0" />
             <geometry>
-                <cylinder radius="0.52" length="0.72"/>
+                <cylinder radius="0.052" length="0.072"/>
             </geometry>
         </visual>
@@ -90,5 +90,5 @@
             <origin xyz="0.0 0.0 0.0" rpy="0.0 0.0 0.0" />
             <geometry>
-                <cylinder radius="0.52" length="0.72"/>
+                <cylinder radius="0.052" length="0.072"/>
             </geometry>
         </collision>

Commit message: fixed wheels

File: src/navvis_description/urdf/robot.xacro (robot description, xacro)
@@ -101,5 +101,5 @@
             <child link="wheel_${side}" />
             <!-- Weirdness with evaluating pi-->
-            <origin xyz="-0.1 ${reflect * .4} 0" r="${-pi/2}" />
+            <origin xyz="-0.1 ${reflect * .4} 0" rpy="${-pi/2} 0 0" />
         </joint>
         <link name="wheel_${side}">
@@ -125,5 +125,5 @@
             <child link="wheel_center" />
             <!-- Weirdness with evaluating pi-->
-            <origin xyz="0.1 0 0" r="${-pi/2}" />
+            <origin xyz="0.1 0 0" rpy="${-pi/2} 0 0" />
         </joint>
         <link name="wheel_center">
